Commit message: Adding laser sensors, contact information and more customisation.

File: catkin_ws_src/pioneer3at_simulation/urdf/pioneer3at.urdf.xacro (robot description, xacro)
@@ -1,4 +1,6 @@
 <?xml version="1.0"?>
 <robot xmlns:sensor="http://playerstage.sourceforge.net/gazebo/xmlschema/#sensor" xmlns:controller="http://playerstage.sourceforge.net/gazebo/xmlschema/#controller" xmlns:interface="http://playerstage.sourceforge.net/gazebo/xmlschema/#interface" xmlns:xacro="http://ros.org/wiki/xacro" name="pioneer3at">
+  <xacro:property name="PI" value="3.141592654" />
+  <xacro:property name="robot_name" value="pioneer3at" />
   <!-- Chassis -->
   <link name="base_link">
@@ -279,8 +281,8 @@
       <inertial>
         <!--mass value="1.2"/>
-			<origin xyz="0 0 0"/>
-			<inertia ixx="0.012411765597" ixy="0" ixz="0"
-                                                      iyy="0.015218160428" iyz="0"
-                                                                           izz="0.011763977943"/-->
+  			<origin xyz="0 0 0"/>
+  			<inertia ixx="0.012411765597" ixy="0" ixz="0"
+                                                        iyy="0.015218160428" iyz="0"
+                                                                             izz="0.011763977943"/-->
         <mass value="1.1"/>
         <origin xyz="0 0 0"/>
@@ -318,45 +320,45 @@
     <gazebo reference="p3at_back_${side}_wheel">
         <sensor name="cb_${side}" type='contact'>
-        <contact>
-        <collision>p3at_back_${side}_wheel_collision</collision>
-        </contact>
+          <contact>
+            <collision>p3at_back_${side}_wheel_collision</collision>
+          </contact>
         </sensor>
-      <kp>1000000.0</kp>
-      <!-- kp and kd for rubber -->
-      <kd>100.0</kd>
-      <mu1>0.9</mu1>
-      <!-- was 10 -->
-      <mu2>0.9</mu2>
-      <!-- how to get these into <surface><friction><ode>... ?
-        slip1 0.5 /slip1
-         slip2 0 /slip2
-      -->
-      <!-- fdir1 0 1 0 /fdir1 -->
-      <!-- see http://github.com/MobileRobots/simulate_traversability-ros-config/issues/6 -->
-      <maxVel>0.0</maxVel>
-      <minDepth>0.001</minDepth>
-      <material value="Gazebo/Black"/>
+        <kp>1000000.0</kp>
+        <!-- kp and kd for rubber -->
+        <kd>100.0</kd>
+        <mu1>0.9</mu1>
+        <!-- was 10 -->
+        <mu2>0.9</mu2>
+        <!-- how to get these into <surface><friction><ode>... ?
+          slip1 0.5 /slip1
+           slip2 0 /slip2
+        -->
+        <!-- fdir1 0 1 0 /fdir1 -->
+        <!-- see http://github.com/MobileRobots/simulate_traversability-ros-config/issues/6 -->
+        <maxVel>0.0</maxVel>
+        <minDepth>0.001</minDepth>
+        <material value="Gazebo/Black"/>
     </gazebo>
     <gazebo reference="p3at_front_${side}_wheel">
         <sensor name="cf_${side}" type='contact'>
-        <contact>
-        <collision>p3at_front_${side}_wheel_collision</collision>
-        </contact>
+          <contact>
+            <collision>p3at_front_${side}_wheel_collision</collision>
+          </contact>
         </sensor>
-      <kp>1000000.0</kp>
-      <!-- kp and kd for rubber -->
-      <kd>100.0</kd>
-      <mu1>0.9</mu1>
-      <!-- was 10 -->
-      <mu2>0.9</mu2>
-      <!-- how to get these into <surface><friction><ode>... ?
-        slip1 0.5 /slip1
-         slip2 0 /slip2
-      -->
-      <!-- fdir1 0 1 0 /fdir1 -->
-      <!-- see http://github.com/MobileRobots/simulate_traversability-ros-config/issues/6 -->
-      <maxVel>0.0</maxVel>
-      <minDepth>0.001</minDepth>
-      <material value="Gazebo/Black"/>
+        <kp>1000000.0</kp>
+        <!-- kp and kd for rubber -->
+        <kd>100.0</kd>
+        <mu1>0.9</mu1>
+        <!-- was 10 -->
+        <mu2>0.9</mu2>
+        <!-- how to get these into <surface><friction><ode>... ?
+          slip1 0.5 /slip1
+           slip2 0 /slip2
+        -->
+        <!-- fdir1 0 1 0 /fdir1 -->
+        <!-- see http://github.com/MobileRobots/simulate_traversability-ros-config/issues/6 -->
+        <maxVel>0.0</maxVel>
+        <minDepth>0.001</minDepth>
+        <material value="Gazebo/Black"/>
     </gazebo>
   </xacro:macro>
@@ -372,5 +374,5 @@
           <origin xyz="0 0 0" rpy="0 0 0"/>
           <geometry>
-            <box size="0.05 0.05 0.05"/>
+            <box size="0.025 0.025 0.025"/>
           </geometry>
         </collision>
@@ -378,5 +380,5 @@
           <origin xyz="0 0 0" rpy="0 0 0"/>
           <geometry>
-            <box size="0.05 0.05 0.05"/>
+            <box size="0.025 0.025 0.025"/>
           </geometry>
           <material name="red"/>
@@ -393,5 +395,5 @@
         <update_rate>30.0</update_rate>
         <camera name="camera_${name}">
-          <pose> 0.05 0 0 0 0 0</pose>
+          <pose> 0.025 0 0 0 0 0</pose>
           <horizontal_fov>${h_fov}</horizontal_fov>
           <image>
@@ -416,8 +418,8 @@
           <alwaysOn>true</alwaysOn>
           <updateRate>0.0</updateRate>
-          <cameraName>pioneer3at/camera_${name}</cameraName>
+          <cameraName>/${robot_name}/camera_${name}</cameraName>
           <imageTopicName>image_raw</imageTopicName>
           <cameraInfoTopicName>camera_info</cameraInfoTopicName>
-          <frameName>camera_${name}</frameName>
+          <frameName>camera_${name}_link</frameName>
           <hackBaseline>0.07</hackBaseline>
           <distortionK1>0.0</distortionK1>
@@ -430,4 +432,68 @@
     </gazebo>
   </xacro:macro>
+  <xacro:macro name="custom_laser" params="name color x y z roll pitch yaw samples resolution min_angle max_angle min_range max_range range_resolution">
+    <joint name="laser_${name}_joint" type="fixed">
+      <axis xyz = "1 0 0"/>
+      <origin xyz="${x} ${y} ${z}" rpy="${roll} ${pitch} ${yaw}"/>
+      <parent link="top_plate"/>
+      <child link="laser_${name}_link"/>
+    </joint>
+    <link name="laser_${name}_link">
+        <collision>
+          <origin xyz="0 0 0" rpy="0 0 0"/>
+          <geometry>
+            <box size="0.025 0.025 0.025"/>
+          </geometry>
+        </collision>
+        <visual>
+          <origin xyz="0 0 0" rpy="0 0 0"/>
+          <geometry>
+            <box size="0.025 0.025 0.025"/>
+          </geometry>
+          <material name="red"/>
+        </visual>
+        <inertial>
+          <mass value="1e-5" />
+          <origin xyz="0 0 0" rpy="0 0 0"/>
+          <inertia ixx="1e-6" ixy="0" ixz="0" iyy="1e-6" iyz="0" izz="1e-6" />
+        </inertial>
+    </link>
+    <gazebo reference="laser_${name}_link">
+        <material value="Gazebo/${color}"/>
+        <sensor type="gpu_ray" name="laser_${name}">
+          <pose>0 0 0 0 0 0</pose>
+          <visualize>true</visualize>
+          <update_rate>40</update_rate>
+          <ray>
+            <scan>
+              <horizontal>
+                <samples>${samples}</samples> <!-- 720 -->
+                <resolution>${resolution}</resolution> <!-- 1 -->
+                <min_angle>${min_angle}</min_angle> <!-- minus 1.570796 -->
+                <max_angle>${max_angle}</max_angle> <!-- 1.570796 -->
+              </horizontal>
+            </scan>
+            <range>
+              <min>${min_range}</min> <!-- 0.10 -->
+              <max>${max_range}</max> <!-- 30.0 -->
+              <resolution>${range_resolution}</resolution> <!-- 0.01 -->
+            </range>
+            <noise>
+              <type>gaussian</type>
+              <!-- Noise parameters based on published spec for Hokuyo laser
+                   achieving "+-30mm" accuracy at range < 10m.  A mean of 0.0m and
+                   stddev of 0.01m will put 99.7% of samples within 0.03m of the true
+                   reading. -->
+              <mean>0.0</mean>
+              <stddev>0.01</stddev>
+            </noise>
+          </ray>
+          <plugin name="gazebo_ros_head_hokuyo_controller" filename="libgazebo_ros_gpu_laser.so">
+            <topicName>/${robot_name}/laser_${name}/scan</topicName>
+            <frameName>laser_${name}_link</frameName>
+          </plugin>
+        </sensor>
+      </gazebo>
+  </xacro:macro>
   <xacro:macro name="p3at_gazebo_ext">
     <gazebo>
@@ -435,5 +501,5 @@
       <plugin name="skid_steer_drive_controller" filename="libgazebo_ros_skid_steer_drive_pioneer3at.so">
         <updateRate>100.0</updateRate>
-        <robotNamespace>sim_p3at</robotNamespace>
+        <robotNamespace>${robot_name}</robotNamespace>
         <leftFrontJoint>p3at_front_left_wheel_joint</leftFrontJoint>
         <rightFrontJoint>p3at_front_right_wheel_joint</rightFrontJoint>
@@ -448,14 +514,35 @@
         <odometryTopic>odom</odometryTopic>
         <odometryFrame>odom</odometryFrame>
-        <broadcastTF>1</broadcastTF>
+        <broadcastTF>false</broadcastTF>
       </plugin>
     </gazebo>
   </xacro:macro>
+  <xacro:macro name="p3at_gazebo_contacts">
+    <gazebo>
+      <plugin name="gazeboRosPioneer3ATContacts" filename="libgazeboRosPioneer3ATContacts.so">
+        <robotNamespace>${robot_name}</robotNamespace>
+        <jointName>p3at_front_left_wheel_joint, p3at_front_right_wheel_joint, p3at_back_left_wheel_joint, p3at_back_right_wheel_joint</jointName>
+        <linkName>p3at_front_left_wheel, p3at_front_right_wheel, p3at_back_left_wheel, p3at_back_right_wheel, base_link</linkName>
+        <updateRate>100.0</updateRate>
+        <alwaysOn>true</alwaysOn>
+        <useROSTime>false</useROSTime>
+        <publishPoseAndTwist>true</publishPoseAndTwist>
+      </plugin>
+    </gazebo>
+  </xacro:macro>
+  <!-- RGB cameras -->
+  <xacro:custom_camera name="one" color="Red" x="0.24" y="0" z="0.04" roll="0" pitch="0.0" yaw="0" h_fov="1.3962634" width="800" height="800" near="0.02" far="100"/>
+  <xacro:custom_camera name="two" color="Blue" x="0.22" y="0.09" z="0.015" roll="0.2" pitch="0.1" yaw="-0.1" h_fov="1.3962634" width="800" height="800" near="0.02" far="100"/>
+  <xacro:custom_camera name="three" color="Yellow" x="0.22" y="-0.1" z="0.015" roll="-0.2" pitch="0.1" yaw="0.2" h_fov="1.3962634" width="800" height="800" near="0.02" far="100"/>
+  <!-- 'RGB' downward sensor -->
+  <xacro:custom_camera name="down" color="White" x="0.0" y="0.0" z="-0.17" roll="0.0" pitch="1.57" yaw="0.0" h_fov="1.0" width="100" height="100" near="0.01" far="1.0"/>
+  <!-- laser sensors -->
+  <xacro:custom_laser name="one" color="White" x="0.24" y="0" z="0.014" roll="0" pitch="0" yaw="0" samples="50" resolution="1" min_angle="${-PI/6}" max_angle="${PI/6}" min_range="0.10" max_range="5.0" range_resolution="0.01"/>
+  <xacro:custom_laser name="two" color="White" x="-0.22" y="0" z="0.014" roll="0" pitch="0" yaw="${PI}" samples="50" resolution="1" min_angle="${-PI/6}" max_angle="${PI/6}" min_range="0.10" max_range="5.0" range_resolution="0.01"/>
+  <!-- skid steer controller -->
   <xacro:p3at_drive_side side="left" reflect="1"/>
   <xacro:p3at_drive_side side="right" reflect="-1"/>
-  <xacro:custom_camera name="one" color="Red" x="0.22" y="0" z="0.02" roll="0" pitch="0" yaw="0" h_fov="1.3962634" width="800" height="800" near="0.02" far="100"/>
-  <xacro:custom_camera name="two" color="Blue" x="0.20" y="0.09" z="0.02" roll="0.2" pitch="0.1" yaw="-0.1" h_fov="1.3962634" width="800" height="800" near="0.02" far="100"/>
-  <xacro:custom_camera name="three" color="Yellow" x="0.20" y="-0.1" z="0.015" roll="-0.2" pitch="0.1" yaw="0.2" h_fov="1.3962634" width="800" height="800" near="0.02" far="100"/>
-  <xacro:custom_camera name="down" color="White" x="0.0" y="0.0" z="-0.17" roll="0.0" pitch="1.57" yaw="0.0" h_fov="1.0" width="100" height="100" near="0.01" far="1"/>
   <xacro:p3at_gazebo_ext/>
+  <!-- contacts and extra robot_state -->
+  <xacro:p3at_gazebo_contacts/>
 </robot>
