Commit message: code to generate textures changed

File: urdf/pioneer3at.urdf.xacro (robot description, xacro)
@@ -1,548 +1,559 @@
 <?xml version="1.0"?>
-<robot xmlns:sensor="http://playerstage.sourceforge.net/gazebo/xmlschema/#sensor" xmlns:controller="http://playerstage.sourceforge.net/gazebo/xmlschema/#controller" xmlns:interface="http://playerstage.sourceforge.net/gazebo/xmlschema/#interface" xmlns:xacro="http://ros.org/wiki/xacro" name="pioneer3at">
-  <xacro:property name="PI" value="3.141592654" />
-  <xacro:property name="robot_name" value="pioneer3at" />
-  <!-- Chassis -->
-  <link name="base_link">
-    <!--  For pointers on inertial and gazebo-related parameters see
-		       * http://wiki.ros.org/urdf/Tutorials/Adding%20Physical%20and%20Collision%20Properties%20to%20a%20URDF%20Model
-                       * http://answers.gazebosim.org/question/4372/the-inertia-matrix-explained/
-		       * http://gazebosim.org/tutorials?tut=inertia&cat=build_robot, and
-                       * http://gazebosim.org/tutorials/?tut=ros_urdf
-                       * http://en.wikipedia.org/wiki/List_of_moment_of_inertia_tensors
-                -->
-    <inertial>
-      <mass value="21"/>
-      <!-- P3AT 18.6kg plus three batteries @ 2.4kg each  minus four wheels @ 1.4 kg ea and top plate @ 0.1 kg-->
-      <origin xyz="0 0 0.177"/>
-      <!--inertia ixx="0.3338" ixy="0.0" ixz="0.0" iyy="0.4783" iyz="0.0" izz="0.3338"/-->
-      <inertia ixx="0.147116667" ixy="0.0" ixz="0.0" iyy="0.334951167" iyz="0.0" izz="0.3978345"/>
-    </inertial>
-    <visual>
-      <origin xyz="0 0 0.177" rpy="0 0 0"/>
-      <geometry name="pioneer_geom">
-        <mesh filename="package://pioneer3at_simulation/meshes/chassis.stl"/>
-      </geometry>
-      <material name="ChassisRed">
-        <color rgba="0.851 0.0 0.0 1.0"/>
-      </material>
-    </visual>
-    <collision>
-      <origin xyz="0 0 0.177" rpy="0 0 0"/>
-      <geometry>
-        <mesh filename="package://pioneer3at_simulation/meshes/chassis.stl"/>
-      </geometry>
-    </collision>
-  </link>
-  <gazebo reference="base_link">
-    <material value="Gazebo/Red"/>
-    <sensor name="blc" type='contact'>
-        <contact>
-        <collision>base_link_collision</collision>
-        </contact>
-    </sensor>
-  </gazebo>
-  <!-- Top -->
-  <link name="top_plate">
-    <!--inertial>
-			<mass value="0.1"/>
-			<origin xyz="-0.025 0 -0.223"/>
-			<inertia ixx="0.01" ixy="0.0" ixz="0.0"
-				 iyy="0.01" iyz="0.0"
- 				izz="0.01"/>
-		</inertial-->
-    <visual>
-      <origin xyz="0 0 0" rpy="0 0 0"/>
-      <geometry name="pioneer_geom">
-        <mesh filename="package://pioneer3at_simulation/meshes/top.stl"/>
-      </geometry>
-      <material name="TopBlack">
-        <color rgba="0.038 0.038 0.038 1.0"/>
-      </material>
-    </visual>
-  </link>
-  <gazebo reference="top_plate">
-    <material>Gazebo/Black</material>
-    <sensor name="tpc" type='contact'>
-        <contact>
-        <collision>top_plate_collision</collision>
-        </contact>
-    </sensor>
-  </gazebo>
-  <joint name="base_top_joint" type="fixed">
-    <origin xyz="0.003 0 0.274" rpy="0 0 0"/>
-    <parent link="base_link"/>
-    <child link="top_plate"/>
-  </joint>
-  <!-- Front + Back Sonar -->
-  <link name="front_sonar">
-    <!--inertial>
-			<mass value="0.1"/>
-			<origin xyz="0 0 0"/>
-			<inertia ixx="0.01" ixy="0.0" ixz="0.0"
-				 iyy="0.01" iyz="0.0" izz="0.01"/>
-		</inertial-->
-    <visual>
-      <origin xyz="0 0 0" rpy="0 0 0"/>
-      <geometry name="pioneer_geom">
-        <mesh filename="package://pioneer3at_simulation/meshes/front_sonar.stl"/>
-      </geometry>
-      <material name="SonarYellow">
-        <color rgba="0.715 0.583 0.210 1.0"/>
-      </material>
-    </visual>
-  </link>
-  <gazebo reference="front_sonar">
-    <material value="Gazebo/Yellow"/>
-  </gazebo>
-  <joint name="base_front_joint" type="fixed">
-    <origin xyz="0.193 0 0.25" rpy="0 0 0"/>
-    <parent link="base_link"/>
-    <child link="front_sonar"/>
-  </joint>
-  <link name="back_sonar">
-    <!--inertial>
-			<mass value="0.1"/>
-			<origin xyz="0 0 0"/>
-			<inertia ixx="0.01" ixy="0.0" ixz="0.0"
-				 iyy="0.01" iyz="0.0" izz="0.01"/>
-		</inertial-->
-    <visual>
-      <origin xyz="0 0 0" rpy="0 0 0"/>
-      <geometry name="pioneer_geom">
-        <mesh filename="package://pioneer3at_simulation/meshes/back_sonar.stl"/>
-      </geometry>
-      <material name="SonarYellow">
-        <color rgba="0.715 0.583 0.210 1.0"/>
-      </material>
-    </visual>
-  </link>
-  <gazebo reference="back_sonar">
-    <material value="Gazebo/Yellow"/>
-  </gazebo>
-  <joint name="base_back_joint" type="fixed">
-    <origin xyz="-0.187 0 0.247" rpy="0 0 0"/>
-    <parent link="base_link"/>
-    <child link="back_sonar"/>
-  </joint>
-  <xacro:macro name="p3at_drive_side" params="side reflect">
-    <!-- Front Axles + Wheels + Hubcaps -->
-    <link name="p3at_front_${side}_axle">
-      <!--inertial>
-			<mass value="0.1"/>
-			<origin xyz="0 0 0"/>
-			<inertia ixx="0.01" ixy="0.0" ixz="0.0"
-				 iyy="0.01" iyz="0.0" izz="0.01"/>
-  	 	</inertial-->
-      <visual>
-        <origin xyz="0 0 0" rpy="0 0 0"/>
-        <geometry name="pioneer_geom">
-          <mesh filename="package://pioneer3at_simulation/meshes/axle.stl"/>
-        </geometry>
-        <material name="AxleGrey">
-          <color rgba="0.5 0.5 0.5 1"/>
-        </material>
-      </visual>
+<robot xmlns:xacro="http://ros.org/wiki/xacro" name="pioneer3at">
+    <xacro:property name="PI" value="3.141592654"/>
+    <xacro:property name="robot_name" value="pioneer3at"/>
+    <!-- Chassis -->
+    <link name="base_link">
+        <!--  For pointers on inertial and gazebo-related parameters see
+                   * http://wiki.ros.org/urdf/Tutorials/Adding%20Physical%20and%20Collision%20Properties%20to%20a%20URDF%20Model
+                           * http://answers.gazebosim.org/question/4372/the-inertia-matrix-explained/
+                   * http://gazebosim.org/tutorials?tut=inertia&cat=build_robot, and
+                           * http://gazebosim.org/tutorials/?tut=ros_urdf
+                           * http://en.wikipedia.org/wiki/List_of_moment_of_inertia_tensors
+                    -->
+        <inertial>
+            <mass value="21"/>
+            <!-- P3AT 18.6kg plus three batteries @ 2.4kg each  minus four wheels @ 1.4 kg ea and top plate @ 0.1 kg-->
+            <origin xyz="0 0 0.177"/>
+            <!--inertia ixx="0.3338" ixy="0.0" ixz="0.0" iyy="0.4783" iyz="0.0" izz="0.3338"/-->
+            <inertia ixx="0.147116667" ixy="0.0" ixz="0.0" iyy="0.334951167" iyz="0.0" izz="0.3978345"/>
+        </inertial>
+        <visual>
+            <origin xyz="0 0 0.177" rpy="0 0 0"/>
+            <geometry name="pioneer_geom">
+                <mesh filename="package://pioneer3at_simulation/meshes/chassis.stl"/>
+            </geometry>
+            <material name="ChassisRed">
+                <color rgba="0.851 0.0 0.0 1.0"/>
+            </material>
+        </visual>
+        <collision>
+            <origin xyz="0 0 0.177" rpy="0 0 0"/>
+            <geometry>
+                <mesh filename="package://pioneer3at_simulation/meshes/chassis.stl"/>
+            </geometry>
+        </collision>
     </link>
-    <gazebo reference="p3at_front_${side}_axle">
-      <material value="Gazebo/Grey"/>
+    <gazebo reference="base_link">
+        <material value="Gazebo/Red"/>
+        <sensor name="blc" type='contact'>
+            <contact>
+                <collision>base_link_collision</collision>
+            </contact>
+        </sensor>
     </gazebo>
-    <joint name="base_front_${side}_axle_joint" type="fixed">
-      <origin xyz="0.135 ${reflect*0.156} 0.111" rpy="0 0 0"/>
-      <parent link="base_link"/>
-      <child link="p3at_front_${side}_axle"/>
+    <!-- Top -->
+    <link name="top_plate">
+        <!--inertial>
+                <mass value="0.1"/>
+                <origin xyz="-0.025 0 -0.223"/>
+                <inertia ixx="0.01" ixy="0.0" ixz="0.0"
+                     iyy="0.01" iyz="0.0"
+                     izz="0.01"/>
+            </inertial-->
+        <visual>
+            <origin xyz="0 0 0" rpy="0 0 0"/>
+            <geometry name="pioneer_geom">
+                <mesh filename="package://pioneer3at_simulation/meshes/top.stl"/>
+            </geometry>
+            <material name="TopBlack">
+                <color rgba="0.038 0.038 0.038 1.0"/>
+            </material>
+        </visual>
+    </link>
+    <gazebo reference="top_plate">
+        <material>Gazebo/Black</material>
+        <sensor name="tpc" type='contact'>
+            <contact>
+                <collision>top_plate_collision</collision>
+            </contact>
+        </sensor>
+    </gazebo>
+    <joint name="base_top_joint" type="fixed">
+        <origin xyz="0.003 0 0.274" rpy="0 0 0"/>
+        <parent link="base_link"/>
+        <child link="top_plate"/>
     </joint>
-    <link name="p3at_front_${side}_hub">
-      <inertial>
-        <mass value="0.1"/>
-        <origin xyz="0 0 0"/>
-        <inertia ixx="0.01" ixy="0.0" ixz="0.0" iyy="0.01" iyz="0.0" izz="0.01"/>
-      </inertial>
-      <visual>
-        <origin xyz="0 0 0" rpy="0 0 0"/>
-        <geometry name="pioneer_geom">
-          <mesh filename="package://pioneer3at_simulation/meshes/${side}_hubcap.stl"/>
-        </geometry>
-        <material name="HubcapYellow">
-          <color rgba="1.0 0.811 0.151 1.0"/>
-        </material>
-      </visual>
+    <!-- Front + Back Sonar -->
+    <link name="front_sonar">
+        <!--inertial>
+                <mass value="0.1"/>
+                <origin xyz="0 0 0"/>
+                <inertia ixx="0.01" ixy="0.0" ixz="0.0"
+                     iyy="0.01" iyz="0.0" izz="0.01"/>
+            </inertial-->
+        <visual>
+            <origin xyz="0 0 0" rpy="0 0 0"/>
+            <geometry name="pioneer_geom">
+                <mesh filename="package://pioneer3at_simulation/meshes/front_sonar.stl"/>
+            </geometry>
+            <material name="SonarYellow">
+                <color rgba="0.715 0.583 0.210 1.0"/>
+            </material>
+        </visual>
     </link>
-    <gazebo reference="p3at_front_${side}_hub">
-      <material value="Gazebo/Yellow"/>
+    <gazebo reference="front_sonar">
+        <material value="Gazebo/Yellow"/>
     </gazebo>
-    <joint name="base_front_${side}_hub_joint" type="fixed">
-      <origin xyz="0 ${reflect*0.041} 0" rpy="0 0 0"/>
-      <parent link="p3at_front_${side}_axle"/>
-      <child link="p3at_front_${side}_hub"/>
+    <joint name="base_front_joint" type="fixed">
+        <origin xyz="0.193 0 0.25" rpy="0 0 0"/>
+        <parent link="base_link"/>
+        <child link="front_sonar"/>
     </joint>
-    <link name="p3at_front_${side}_wheel">
-      <inertial>
-        <!-- 1.4 kg - axle 0.1 kg - hub 0.1 kg -->
-        <!--mass value="1.2"/>
-			<origin xyz="0 0 0"/>
-			<inertia ixx="0.012411765597" ixy="0" ixz="0"
-         iyy="0.015218160428" iyz="0" izz="0.011763977943"/-->
-        <mass value="1.1"/>
-        <origin xyz="0 0 0"/>
-        <!--inertia ixx="0.005240625" ixy="0" ixz="0" iyy="0.009075" iyz="0" izz="0.005240625"/-->
-        <inertia ixx="0.002216042" ixy="0" ixz="0" iyy="0.00397375" iyz="0" izz="0.002216042"/>
-      </inertial>
-      <visual>
-        <origin xyz="0 0 0" rpy="0 0 0"/>
-        <geometry name="pioneer_geom">
-          <mesh filename="package://pioneer3at_simulation/meshes/wheel.stl" scale="0.75 0.66 0.75"/>
-        </geometry>
-        <material name="WheelBlack">
-          <color rgba="0.117 0.117 0.117 1"/>
-        </material>
-      </visual>
-      <collision>
-        <origin xyz="0 0 0" rpy="${-3.1415927/2} 0 0"/>
-        <geometry>
-          <!--mesh filename="package://pioneer3at_simulation/meshes/wheel.stl"/-->
-          <cylinder radius="0.085" length="0.05"/>
-        </geometry>
-      </collision>
+    <link name="back_sonar">
+        <!--inertial>
+                <mass value="0.1"/>
+                <origin xyz="0 0 0"/>
+                <inertia ixx="0.01" ixy="0.0" ixz="0.0"
+                     iyy="0.01" iyz="0.0" izz="0.01"/>
+            </inertial-->
+        <visual>
+            <origin xyz="0 0 0" rpy="0 0 0"/>
+            <geometry name="pioneer_geom">
+                <mesh filename="package://pioneer3at_simulation/meshes/back_sonar.stl"/>
+            </geometry>
+            <material name="SonarYellow">
+                <color rgba="0.715 0.583 0.210 1.0"/>
+            </material>
+        </visual>
     </link>
-    <gazebo reference="p3at_front_${side}_wheel">
-      <material value="Gazebo/Black"/>
+    <gazebo reference="back_sonar">
+        <material value="Gazebo/Yellow"/>
     </gazebo>
-    <joint name="p3at_front_${side}_wheel_joint" type="continuous">
-      <axis xyz="0 1 0"/>
-      <anchor xyz="0 0 0"/>
-      <limit effort="10" velocity="10"/>
-      <joint_properties damping="0.7"/>
-      <origin xyz="0 0 0" rpy="0 0 0"/>
-      <parent link="p3at_front_${side}_hub"/>
-      <child link="p3at_front_${side}_wheel"/>
+    <joint name="base_back_joint" type="fixed">
+        <origin xyz="-0.187 0 0.247" rpy="0 0 0"/>
+        <parent link="base_link"/>
+        <child link="back_sonar"/>
     </joint>
-    <!-- Back Axles + Wheels + Hubcaps -->
-    <link name="p3at_back_${side}_axle">
-      <!--inertial>
-			<mass value="0.1"/>
-			<origin xyz="0 0 0"/>
-			<inertia ixx="0.01" ixy="0.0" ixz="0.0"
-				 iyy="0.01" iyz="0.0" izz="0.01"/>
-  	 	</inertial-->
-      <visual>
-        <origin xyz="0 0 0" rpy="0 0 0"/>
-        <geometry name="pioneer_geom">
-          <mesh filename="package://pioneer3at_simulation/meshes/axle.stl"/>
-        </geometry>
-        <material name="AxleGrey">
-          <color rgba="0.5 0.5 0.5 1"/>
-        </material>
-      </visual>
-      <collision>
-        <origin xyz="0 0 0" rpy="0 0 0"/>
-        <geometry>
-          <mesh filename="package://pioneer3at_simulation/meshes/axle.stl"/>
-        </geometry>
-      </collision>
-    </link>
-    <gazebo reference="p3at_back_${side}_axle">
-      <material value="Gazebo/Grey"/>
-    </gazebo>
-    <joint name="p3at_back_${side}_axle_joint" type="fixed">
-      <origin xyz="-0.134 ${reflect*0.156} 0.111" rpy="0 0 0"/>
-      <parent link="base_link"/>
-      <child link="p3at_back_${side}_axle"/>
-    </joint>
-    <link name="p3at_back_${side}_hub">
-      <inertial>
-        <mass value="0.1"/>
-        <origin xyz="0 0 0"/>
-        <inertia ixx="0.01" ixy="0.0" ixz="0.0" iyy="0.01" iyz="0.0" izz="0.01"/>
-      </inertial>
-      <visual>
-        <origin xyz="0 0 0" rpy="0 0 0"/>
-        <geometry name="pioneer_geom">
-          <mesh filename="package://pioneer3at_simulation/meshes/${side}_hubcap.stl"/>
-        </geometry>
-        <material name="HubcapYellow"/>
-      </visual>
-      <collision>
-        <origin xyz="0 0 0" rpy="0 0 0"/>
-        <geometry>
-          <mesh filename="package://pioneer3at_simulation/meshes/${side}_hubcap.stl"/>
-        </geometry>
-      </collision>
-    </link>
-    <gazebo reference="p3at_back_${side}_hub">
-      <material value="Gazebo/Yellow"/>
-    </gazebo>
-    <joint name="p3at_back_${side}_hub_joint" type="fixed">
-      <origin xyz="-0 ${reflect*0.041} 0" rpy="0 0 0"/>
-      <parent link="p3at_back_${side}_axle"/>
-      <child link="p3at_back_${side}_hub"/>
-    </joint>
-    <link name="p3at_back_${side}_wheel">
-      <inertial>
-        <!--mass value="1.2"/>
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